Commit message: add scene objects

File: urdf/stair.urdf (robot description, URDF)
Before this commit: robot stair_skeleton, 2 links, 1 joints
Links:
- removed link stair_link
- added link base_link
- added link step_1; collision box size=0.4 1.0 0.15; visual box size=0.4 1.0 0.15
- added link step_2_top; collision box size=0.8 1.0 0.30; visual box size=0.8 1.0 0.30
- added link step_3; collision box size=0.4 1.0 0.15; visual box size=0.4 1.0 0.15
Joints:
- removed joint stair_joint
- added joint base_to_step_1: type fixed, parent base_link, child step_1
- added joint base_to_step_2: type fixed, parent base_link, child step_2_top
- added joint base_to_step_3: type fixed, parent base_link, child step_3
- added joint fixed_to_world: type fixed, parent world, child base_link, origin xyz=0.45 0 0 rpy=0 0 0
